Commit message: added end-effector and changed IK solver to ik-trac

File: denso_robot_descriptions/vs6577_description/vs6577.urdf (robot description, URDF)
Before this commit: robot vs6577, 8 links, 7 joints
Links:
- added link vacuum, mass 0.6; collision mesh filename=package://denso_robot_descriptions/tool_description/vs6577_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; visual mesh filename=package://denso_robot_descriptions/tool_description/vs6577_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
Joints:
- added joint tool: type fixed, parent J6, child vacuum, origin xyz=0 0 0.264 rpy=0 0 0
